File: hardware/bitsy-v1.1b/icebreaker-bitsy.kicad_sch (KiCad schematic)
At the start: 95 parts, among them J1 USB_C, P0 0, P1 1, P10 10, P11 11, P12 12, P13 13, P14 14, P15 15, P16 16, P17 17, P18 18, P19 19, P2 2, P20 20, P21 21, P22 22, P23 23, P24 GND, P25 GND, P26 GND, P27 3V3, P28 3V3, P29 VIN, P3 3, P30 CDONE, P31 CRESET, P32 UP, P33 UP, P34 UP, P35 UP, P36 CS, P37 SCK, P38 MISO, P39 MOSI, P4 4, P40 IO3, P41 IO2, P5 5, P6 6, P7 7, P8 8, P9 9, SW1 TACT, U1 USBLC6-2, U2 TLV75533PDRV, U3 TLV73312PDRV, U4 LY68L6400, U5 W25Q128JVxxM, U6 ICE40UP5K-SG48, X1 12MHz

Commit message: Exploring DiffPair Routing
Connections:
- net IOB_8a renamed IOB_DP2+
- net IOB_9b renamed IOB_DP2-
Changed lines of the file:
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@@
     (effects (font (size 1.27 1.27)) (justify left bottom))
   )
-  (label "IOB_8a" (at 177.8 50.8 0)
+  (label "IOB_DP2+" (at 177.8 50.8 0)
     (effects (font (size 1.27 1.27)) (justify left bottom))
   )
-  (label "IOB_9b" (at 177.8 53.34 0)
+  (label "IOB_DP2-" (at 177.8 53.34 0)
     (effects (font (size 1.27 1.27)) (justify left bottom))
   )
